File: corne-cherry.kicad_pcb (KiCad board)
At the start: 2 copper layers, 275.5 x 105.6 mm, 188 parts, among them J1 MJ-4PP-9, J2 OLED, J3 MJ-4PP-9, J4 OLED, SW1 SW_PUSH, SW10 SW_PUSH, SW11 SW_PUSH, SW12 SW_PUSH, SW13 SW_PUSH, SW14 SW_PUSH, SW15 SW_PUSH, SW16 SW_PUSH, SW17 SW_PUSH, SW18 SW_PUSH, SW19 SW_PUSH, SW2 SW_PUSH, SW20 SW_PUSH, SW21 SW_PUSH, SW22 SW_PUSH, SW23 SW_PUSH, SW24 SW_PUSH, SW25 SW_PUSH, SW26 SW_PUSH, SW27 SW_PUSH, SW28 SW_PUSH, SW29 SW_PUSH, SW3 SW_PUSH, SW30 SW_PUSH, SW31 SW_PUSH, SW32 SW_PUSH, SW33 SW_PUSH, SW34 SW_PUSH, SW35 SW_PUSH, SW36 SW_PUSH, SW37 SW_PUSH, SW38 SW_PUSH, SW39 SW_PUSH, SW4 SW_PUSH, SW40 SW_PUSH, SW41 SW_PUSH, SW42 SW_PUSH, SW43 SW_PUSH, SW44 SW_PUSH, SW45 SW_PUSH, SW46 SW_PUSH, SW47 SW_PUSH, SW48 SW_PUSH, SW5 SW_PUSH, SW6 SW_PUSH, SW7 SW_PUSH, SW8 SW_PUSH, SW9 SW_PUSH, U1 ProMicro, U2 ProMicro

Commit message: finished pcb design; minor improvements are still to be expected
Parts:
- removed the REF** at (238.7, 102.5)
- removed the REF** at (278.9, 102.5)
- removed the REF** at (58.1, 102.5)
- removed the REF** at (20.2, 102.5)
- added REF**: Breakaway_Tabs, kbd:Breakaway_Tabs, F.Cu at (130.7, 91.7)
- added REF**: Breakaway_Tabs, kbd:Breakaway_Tabs, B.Cu at (166.0, 91.7)
- moved D19 57.7 mm to (99.8, 85.0), turned to 150 degrees
- moved D21 55.9 mm to (119.2, 89.1), turned to 150 degrees
- moved LED25 53.1 mm to (99.4, 94.1), turned to 60 degrees
- moved SW21 53.1 mm to (114.9, 95.9), turned to 60 degrees
- moved LED27 52.2 mm to (119.0, 98.2), turned to 60 degrees
- moved SW19 50.3 mm to (95.2, 91.7), turned to 60 degrees
- moved D20 37.0 mm to (110.6, 106.4), turned to 150 degrees
- moved SW20 30.2 mm to (106.3, 113.1), turned to 60 degrees
- moved LED26 29.7 mm to (110.5, 115.5), turned to 60 degrees
- moved Ref** 2.86 mm to (139.4, 82.8)
- moved Ref** 2.81 mm to (157.2, 82.8)
- moved Ref** 0.78 mm to (128.5, 74.7)
- moved D12 0.51 mm to (122.7, 51.9)
Routing:
- net GND: track 533.2 -> 667.3 mm, vias 2 -> 12
- net VCC: track 510.2 -> 613.5 mm, vias 2 -> 4
- net col0: track 113.4 -> 193.1 mm, vias 6 -> 8
- net row3: track 131.5 -> 207.7 mm, vias 1 -> 4
- net Net-(LED23-Pad2): track 0.00 -> 59.1 mm, vias 0 -> 4
- net col4: track 83.9 -> 141.5 mm, vias 5 -> 7
- net Net-(LED3-Pad3): track 0.00 -> 49.9 mm, vias 0 -> 2
- net Net-(LED4-Pad2): track 0.00 -> 48.7 mm, vias 0 -> 4
- net col3: track 106.7 -> 152.0 mm, vias 5 -> 7
- net Net-(LED22-Pad4): track 0.00 -> 45.2 mm, vias 0 -> 4
- net Net-(LED17-Pad2): track 0.00 -> 38.9 mm, vias 0 -> 2
- net Net-(LED5-Pad2): track 0.00 -> 33.7 mm, vias 0 -> 2
- net col5: track 62.1 -> 95.1 mm, vias 4 -> 6
- net Net-(LED28-Pad2): track 1.56 -> 33.6 mm, vias 1 -> 2
- net Net-(LED27-Pad4): track 0.00 -> 31.0 mm, vias 0 -> 2
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Other:
- board size 275.5 x 105.6 mm -> 275.5 x 114.5 mm
- board text removed: "Cornetrack Cherry v1.0 PCB Designed by jannikwibker"

Commit message: updated schematic and pcb
schematic: fixed unconnected pins and aligned some components to the grid
pcb: updated wires according to new schematic, created outline (edge
cuts layer), added a few more labels, fixed a few smaller mistakes
Parts:
- moved D46 4.83 mm to (279.4, 92.7)
- moved LED57 4.83 mm to (271.8, 97.6)
- moved SW46 4.83 mm to (271.8, 92.8)
- moved D43 4.83 mm to (27.7, 92.7)
- moved LED55 4.83 mm to (20.1, 97.6)
- moved SW43 4.83 mm to (20.1, 92.8)
- moved Ref** 1.14 mm to (29.7, 45.2)
- moved Ref** 1.02 mm to (128.5, 73.7)
Connections:
- LED1 pad 3: Net-(LED1-Pad3) -> GND
- LED2 pad 3: Net-(LED2-Pad3) -> GND
- LED28 pad 3: Net-(LED28-Pad3) -> GNDA
- LED29 pad 3: Net-(LED29-Pad3) -> GNDA
- LED3 pad 3: Net-(LED3-Pad3) -> GND
- LED30 pad 3: Net-(LED30-Pad3) -> GNDA
- LED31 pad 3: Net-(LED31-Pad3) -> GNDA
- LED33 pad 3: Net-(LED30-Pad3) -> GNDA
- LED4 pad 3: Net-(LED4-Pad3) -> GND
- LED6 pad 3: Net-(LED3-Pad3) -> GND
Routing:
- net GND: track 667.3 -> 725.8 mm, vias 12 -> 22
- net GNDA: track 675.3 -> 726.5 mm, vias 8 -> 17
- net Net-(LED3-Pad3): track 49.9 -> 0.00 mm, vias 2 -> 0
- net Net-(LED30-Pad3): track 49.7 -> 0.00 mm, vias 2 -> 0
- net VDD: track 669.4 -> 661.9 mm
- net row3: track 207.7 -> 212.5 mm
- net Net-(LED46-Pad2): track 28.9 -> 33.7 mm
- net row3_r: track 245.9 -> 241.1 mm
- net col0: track 193.1 -> 189.8 mm
- net col0_r: track 195.0 -> 198.2 mm
- net VCC: track 613.5 -> 610.7 mm
- net Net-(LED19-Pad2): track 25.0 -> 27.0 mm
- net col1: track 171.7 -> 172.2 mm
Other:
- outline, holes or cut-outs redrawn
- board text added: "JLCJLCJLCJLC"
- board text added: "cornetrack pcb - designed by jannikwibker"
- board text added: "https://github.com/JannikWibker"
- board text added: "rev 1.0"
- board text removed: "Cornetrack v1.0 PCB Designed by jannikwibker"

Commit message: added gerber files and added even more lables to the pcb
Other:
- board text added: "LED57"
- board text added: "left pcb"
- board text added: "right pcb"
