File: cornetrack.sch (KiCad schematic (older format))
At the start: 164 parts, among them J1 MJ-4PP-9, J2 OLED, J3 MJ-4PP-9, J4 OLED, SW1 SW_PUSH, SW10 SW_PUSH, SW11 SW_PUSH, SW12 SW_PUSH, SW13 SW_PUSH, SW14 SW_PUSH, SW15 SW_PUSH, SW16 SW_PUSH, SW17 SW_PUSH, SW18 SW_PUSH, SW19 SW_PUSH, SW2 SW_PUSH, SW20 SW_PUSH, SW21 SW_PUSH, SW22 SW_PUSH, SW23 SW_PUSH, SW24 SW_PUSH, SW25 SW_PUSH, SW26 SW_PUSH, SW27 SW_PUSH, SW28 SW_PUSH, SW29 SW_PUSH, SW3 SW_PUSH, SW30 SW_PUSH, SW31 SW_PUSH, SW32 SW_PUSH, SW33 SW_PUSH, SW34 SW_PUSH, SW35 SW_PUSH, SW36 SW_PUSH, SW37 SW_PUSH, SW38 SW_PUSH, SW39 SW_PUSH, SW4 SW_PUSH, SW40 SW_PUSH, SW41 SW_PUSH, SW42 SW_PUSH, SW43 SW_PUSH, SW44 SW_PUSH, SW45 SW_PUSH, SW46 SW_PUSH, SW47 SW_PUSH, SW48 SW_PUSH, SW5 SW_PUSH, SW6 SW_PUSH, SW7 SW_PUSH, SW8 SW_PUSH, SW9 SW_PUSH, U1 ProMicro, U2 ProMicro

Commit message: renamed project, diode rotation, assembly - renamed project from corne-cherry to cornetrack - tried to have all diodes rotated the same way - did numerous assembly related shenanigans; this is all in an attempt to get jlcpcb to properly detect component orientation
Parts:
- D1, D10, D11, D12, D13, D14, D15, D16, D17, D18, D19, D2, D20, D21, D22, D23, D24, D25, D26, D27, D28, D29, D3, D30, D31, D32, D33, D34, D35, D36, D37, D38, D39, D4, D40, D41, D42, D43, D44, D45, D46, D47, D48, D5, D6, D7, D8, D9: LCSC Part # (none) -> C81598
Changed lines of the file:
@@
 encoding utf-8
 Sheet 1 1
-Title "Corne Cherry"
-Date "2020-07-20"
-Rev "3.0"
-Comp "foostan"
-Comment1 ""
+Title "cornetrack"
+Date "2020-09-10"
+Rev "1.0"
+Comp "jannikwibker"
+Comment1 "based on crkbd / corne by foostan"
 Comment2 ""
 Comment3 ""
@@
 F 2 "kbd:D3_SMD_v2" H 12825 1500 50  0001 C CNN
 F 3 "" H 12825 1500 50  0001 C CNN
+F 4 "C81598" H 12825 1500 50  0001 C CNN "LCSC Part #"
 	1    12825 1500
 	0    -1   -1   0
@@
 F 2 "kbd:D3_SMD_v2" H 13525 1500 50  0001 C CNN
 F 3 "" H 13525 1500 50  0001 C CNN
+F 4 "C81598" H 13525 1500 50  0001 C CNN "LCSC Part #"
 	1    13525 1500
 	0    -1   -1   0
@@
 F 2 "kbd:D3_SMD_v2" H 14225 1500 50  0001 C CNN
 F 3 "" H 14225 1500 50  0001 C CNN
+F 4 "C81598" H 14225 1500 50  0001 C CNN "LCSC Part #"
 	1    14225 1500
 	0    -1   -1   0
@@
 F 2 "kbd:D3_SMD_v2" H 14925 1500 50  0001 C CNN
 F 3 "" H 14925 1500 50  0001 C CNN
+F 4 "C81598" H 14925 1500 50  0001 C CNN "LCSC Part #"
 	1    14925 1500
 	0    -1   -1   0
@@
 F 2 "kbd:D3_SMD_v2" H 15625 1500 50  0001 C CNN
 F 3 "" H 15625 1500 50  0001 C CNN
+F 4 "C81598" H 15625 1500 50  0001 C CNN "LCSC Part #"
 	1    15625 1500
 	0    -1   -1   0
@@
 F 2 "kbd:D3_SMD_v2" H 12125 1500 50  0001 C CNN
 F 3 "" H 12125 1500 50  0001 C CNN
+F 4 "C81598" H 12125 1500 50  0001 C CNN "LCSC Part #"
 	1    12125 1500
 	0    -1   -1   0
@@
 F 2 "kbd:D3_SMD_v2" H 12825 2100 50  0001 C CNN
 F 3 "" H 12825 2100 50  0001 C CNN
+F 4 "C81598" H 12825 2100 50  0001 C CNN "LCSC Part #"
 	1    12825 2100
 	0    -1   -1   0
@@
 F 2 "kbd:D3_SMD_v2" H 13525 2100 50  0001 C CNN
 F 3 "" H 13525 2100 50  0001 C CNN
+F 4 "C81598" H 13525 2100 50  0001 C CNN "LCSC Part #"
 	1    13525 2100
 	0    -1   -1   0
@@
 F 2 "kbd:D3_SMD_v2" H 14225 2100 50  0001 C CNN
 F 3 "" H 14225 2100 50  0001 C CNN
+F 4 "C81598" H 14225 2100 50  0001 C CNN "LCSC Part #"
 	1    14225 2100
 	0    -1   -1   0
@@
 F 2 "kbd:D3_SMD_v2" H 14925 2100 50  0001 C CNN
 F 3 "" H 14925 2100 50  0001 C CNN
+F 4 "C81598" H 14925 2100 50  0001 C CNN "LCSC Part #"
 	1    14925 2100
 	0    -1   -1   0
@@
 F 2 "kbd:D3_SMD_v2" H 12125 2100 50  0001 C CNN
 F 3 "" H 12125 2100 50  0001 C CNN
+F 4 "C81598" H 12125 2100 50  0001 C CNN "LCSC Part #"
 	1    12125 2100
 	0    -1   -1   0
@@
 F 2 "kbd:D3_SMD_v2" H 12825 2700 50  0001 C CNN
 F 3 "" H 12825 2700 50  0001 C CNN
+F 4 "C81598" H 12825 2700 50  0001 C CNN "LCSC Part #"
 	1    12825 2700
 	0    -1   -1   0
@@
 F 2 "kbd:D3_SMD_v2" H 13525 2700 50  0001 C CNN
 F 3 "" H 13525 2700 50  0001 C CNN
+F 4 "C81598" H 13525 2700 50  0001 C CNN "LCSC Part #"
 	1    13525 2700
 	0    -1   -1   0
@@
 F 2 "kbd:D3_SMD_v2" H 14225 2700 50  0001 C CNN
 F 3 "" H 14225 2700 50  0001 C CNN
+F 4 "C81598" H 14225 2700 50  0001 C CNN "LCSC Part #"
 	1    14225 2700
 	0    -1   -1   0
@@
 F 2 "kbd:D3_SMD_v2" H 14925 2700 50  0001 C CNN
 F 3 "" H 14925 2700 50  0001 C CNN
+F 4 "C81598" H 14925 2700 50  0001 C CNN "LCSC Part #"
 	1    14925 2700
 	0    -1   -1   0
@@
 F 2 "kbd:D3_SMD_v2" H 15625 2700 50  0001 C CNN
 F 3 "" H 15625 2700 50  0001 C CNN
+F 4 "C81598" H 15625 2700 50  0001 C CNN "LCSC Part #"
 	1    15625 2700
 	0    -1   -1   0
@@
 F 2 "kbd:D3_SMD_v2" H 12125 2700 50  0001 C CNN
 F 3 "" H 12125 2700 50  0001 C CNN
+F 4 "C81598" H 12125 2700 50  0001 C CNN "LCSC Part #"
 	1    12125 2700
 	0    -1   -1   0
@@
 F 2 "kbd:D3_SMD_v2" H 14925 3300 50  0001 C CNN
 F 3 "" H 14925 3300 50  0001 C CNN
+F 4 "C81598" H 14925 3300 50  0001 C CNN "LCSC Part #"
 	1    14925 3300
 	0    -1   -1   0
@@
 F 2 "kbd:D3_SMD_v2" H 15625 3300 50  0001 C CNN
 F 3 "" H 15625 3300 50  0001 C CNN
+F 4 "C81598" H 15625 3300 50  0001 C CNN "LCSC Part #"
 	1    15625 3300
 	0    -1   -1   0
@@
 F 2 "kbd:D3_SMD_v2" H 12125 3300 50  0001 C CNN
 F 3 "" H 12125 3300 50  0001 C CNN
+F 4 "C81598" H 12125 3300 50  0001 C CNN "LCSC Part #"
 	1    12125 3300
 	0    -1   -1   0
@@
 F 2 "kbd:D3_SMD_v2" H 14225 3300 50  0001 C CNN
 F 3 "" H 14225 3300 50  0001 C CNN
+F 4 "C81598" H 14225 3300 50  0001 C CNN "LCSC Part #"
 	1    14225 3300
 	0    -1   -1   0
@@
 F 2 "kbd:D3_SMD_v2" H 12825 3300 50  0001 C CNN
 F 3 "" H 12825 3300 50  0001 C CNN
+F 4 "C81598" H 12825 3300 50  0001 C CNN "LCSC Part #"
 	1    12825 3300
 	0    -1   -1   0
@@
 F 2 "kbd:D3_SMD_v2" H 13525 3300 50  0001 C CNN
 F 3 "" H 13525 3300 50  0001 C CNN
+F 4 "C81598" H 13525 3300 50  0001 C CNN "LCSC Part #"
 	1    13525 3300
 	0    -1   -1   0
@@
 F 2 "kbd:D3_SMD_v2" H 15625 2100 50  0001 C CNN
 F 3 "" H 15625 2100 50  0001 C CNN
+F 4 "C81598" H 15625 2100 50  0001 C CNN "LCSC Part #"
 	1    15625 2100
 	0    -1   -1   0
@@
 F 2 "kbd:D3_SMD_v2" H 4900 1475 50  0001 C CNN
 F 3 "" H 4900 1475 50  0001 C CNN
+F 4 "C81598" H 4900 1475 50  0001 C CNN "LCSC Part #"
 	1    4900 1475
 	0    -1   -1   0
@@
 F 2 "kbd:D3_SMD_v2" H 5600 1475 50  0001 C CNN
 F 3 "" H 5600 1475 50  0001 C CNN
+F 4 "C81598" H 5600 1475 50  0001 C CNN "LCSC Part #"
 	1    5600 1475
 	0    -1   -1   0
@@
 F 2 "kbd:D3_SMD_v2" H 6300 1475 50  0001 C CNN
 F 3 "" H 6300 1475 50  0001 C CNN
+F 4 "C81598" H 6300 1475 50  0001 C CNN "LCSC Part #"
 	1    6300 1475
 	0    -1   -1   0
@@
 F 2 "kbd:D3_SMD_v2" H 7000 1475 50  0001 C CNN
 F 3 "" H 7000 1475 50  0001 C CNN
+F 4 "C81598" H 7000 1475 50  0001 C CNN "LCSC Part #"
 	1    7000 1475
 	0    -1   -1   0
@@
 F 2 "kbd:D3_SMD_v2" H 7700 1475 50  0001 C CNN
 F 3 "" H 7700 1475 50  0001 C CNN
+F 4 "C81598" H 7700 1475 50  0001 C CNN "LCSC Part #"
 	1    7700 1475
 	0    -1   -1   0
@@
 F 2 "kbd:D3_SMD_v2" H 4200 1475 50  0001 C CNN
 F 3 "" H 4200 1475 50  0001 C CNN
+F 4 "C81598" H 4200 1475 50  0001 C CNN "LCSC Part #"
 	1    4200 1475
 	0    -1   -1   0
@@
 F 2 "kbd:D3_SMD_v2" H 4900 2075 50  0001 C CNN
 F 3 "" H 4900 2075 50  0001 C CNN
+F 4 "C81598" H 4900 2075 50  0001 C CNN "LCSC Part #"
 	1    4900 2075
 	0    -1   -1   0
@@
 F 2 "kbd:D3_SMD_v2" H 5600 2075 50  0001 C CNN
 F 3 "" H 5600 2075 50  0001 C CNN
+F 4 "C81598" H 5600 2075 50  0001 C CNN "LCSC Part #"
 	1    5600 2075
 	0    -1   -1   0
@@
 F 2 "kbd:D3_SMD_v2" H 6300 2075 50  0001 C CNN
 F 3 "" H 6300 2075 50  0001 C CNN
+F 4 "C81598" H 6300 2075 50  0001 C CNN "LCSC Part #"
 	1    6300 2075
 	0    -1   -1   0
@@
 F 2 "kbd:D3_SMD_v2" H 7000 2075 50  0001 C CNN
 F 3 "" H 7000 2075 50  0001 C CNN
+F 4 "C81598" H 7000 2075 50  0001 C CNN "LCSC Part #"
 	1    7000 2075
 	0    -1   -1   0
@@
 F 2 "kbd:D3_SMD_v2" H 7700 2075 50  0001 C CNN
 F 3 "" H 7700 2075 50  0001 C CNN
+F 4 "C81598" H 7700 2075 50  0001 C CNN "LCSC Part #"
 	1    7700 2075
 	0    -1   -1   0
@@
 F 2 "kbd:D3_SMD_v2" H 4200 2075 50  0001 C CNN
 F 3 "" H 4200 2075 50  0001 C CNN
+F 4 "C81598" H 4200 2075 50  0001 C CNN "LCSC Part #"
 	1    4200 2075
 	0    -1   -1   0
@@
 F 2 "kbd:D3_SMD_v2" H 4900 2675 50  0001 C CNN
 F 3 "" H 4900 2675 50  0001 C CNN
+F 4 "C81598" H 4900 2675 50  0001 C CNN "LCSC Part #"
 	1    4900 2675
 	0    -1   -1   0
@@
 F 2 "kbd:D3_SMD_v2" H 5600 2675 50  0001 C CNN
 F 3 "" H 5600 2675 50  0001 C CNN
+F 4 "C81598" H 5600 2675 50  0001 C CNN "LCSC Part #"
 	1    5600 2675
 	0    -1   -1   0
@@
 F 2 "kbd:D3_SMD_v2" H 6300 2675 50  0001 C CNN
 F 3 "" H 6300 2675 50  0001 C CNN
+F 4 "C81598" H 6300 2675 50  0001 C CNN "LCSC Part #"
 	1    6300 2675
 	0    -1   -1   0
@@
 F 2 "kbd:D3_SMD_v2" H 7000 2675 50  0001 C CNN
 F 3 "" H 7000 2675 50  0001 C CNN
+F 4 "C81598" H 7000 2675 50  0001 C CNN "LCSC Part #"
 	1    7000 2675
 	0    -1   -1   0
@@
 F 2 "kbd:D3_SMD_v2" H 7000 3275 50  0001 C CNN
 F 3 "" H 7000 3275 50  0001 C CNN
+F 4 "C81598" H 7000 3275 50  0001 C CNN "LCSC Part #"
 	1    7000 3275
 	0    -1   -1   0
@@
 F 2 "kbd:D3_SMD_v2" H 7700 3275 50  0001 C CNN
 F 3 "" H 7700 3275 50  0001 C CNN
+F 4 "C81598" H 7700 3275 50  0001 C CNN "LCSC Part #"
 	1    7700 3275
 	0    -1   -1   0
@@
 F 2 "kbd:D3_SMD_v2" H 6300 3275 50  0001 C CNN
 F 3 "" H 6300 3275 50  0001 C CNN
+F 4 "C81598" H 6300 3275 50  0001 C CNN "LCSC Part #"
 	1    6300 3275
 	0    -1   -1   0
@@
 F 2 "kbd:D3_SMD_v2" H 4200 2675 50  0001 C CNN
 F 3 "" H 4200 2675 50  0001 C CNN
+F 4 "C81598" H 4200 2675 50  0001 C CNN "LCSC Part #"
 	1    4200 2675
 	0    -1   -1   0
@@
 F 2 "kbd:D3_SMD_v2" H 4200 3275 50  0001 C CNN
 F 3 "" H 4200 3275 50  0001 C CNN
+F 4 "C81598" H 4200 3275 50  0001 C CNN "LCSC Part #"
 	1    4200 3275
 	0    -1   -1   0
@@
 F 2 "kbd:D3_SMD_v2" H 4900 3275 50  0001 C CNN
 F 3 "" H 4900 3275 50  0001 C CNN
+F 4 "C81598" H 4900 3275 50  0001 C CNN "LCSC Part #"
 	1    4900 3275
 	0    -1   -1   0
@@
 F 2 "kbd:D3_SMD_v2" H 5600 3275 50  0001 C CNN
 F 3 "" H 5600 3275 50  0001 C CNN
+F 4 "C81598" H 5600 3275 50  0001 C CNN "LCSC Part #"
 	1    5600 3275
 	0    -1   -1   0
@@
 F 2 "kbd:D3_SMD_v2" H 7700 2675 50  0001 C CNN
 F 3 "" H 7700 2675 50  0001 C CNN
+F 4 "C81598" H 7700 2675 50  0001 C CNN "LCSC Part #"
 	1    7700 2675
 	0    -1   -1   0
