File: jade/cornetrack.kicad_pcb (KiCad board)
At the start: 2 copper layers, 539 x 198.5 mm, 222 parts, among them J1 MJ-4PP-9, J2 OLED, J3 MJ-4PP-9, J4 OLED, SW1 SW_PUSH, SW10 SW_PUSH, SW11 SW_PUSH, SW12 SW_PUSH, SW13 SW_PUSH, SW14 SW_PUSH, SW15 SW_PUSH, SW16 SW_PUSH, SW17 SW_PUSH, SW18 SW_PUSH, SW19 SW_PUSH, SW2 SW_PUSH, SW20 SW_PUSH, SW21 SW_PUSH, SW22 SW_PUSH, SW23 SW_PUSH, SW24 SW_PUSH, SW25 SW_PUSH, SW26 SW_PUSH, SW27 SW_PUSH, SW28 SW_PUSH, SW29 SW_PUSH, SW3 SW_PUSH, SW30 SW_PUSH, SW31 SW_PUSH, SW32 SW_PUSH, SW33 SW_PUSH, SW34 SW_PUSH, SW35 SW_PUSH, SW36 SW_PUSH, SW37 SW_PUSH, SW38 SW_PUSH, SW39 SW_PUSH, SW4 SW_PUSH, SW40 SW_PUSH, SW41 SW_PUSH, SW42 SW_PUSH, SW43 SW_PUSH, SW44 SW_PUSH, SW45 SW_PUSH, SW46 SW_PUSH, SW47 SW_PUSH, SW48 SW_PUSH, SW5 SW_PUSH, SW6 SW_PUSH, SW7 SW_PUSH, SW8 SW_PUSH, SW9 SW_PUSH, U1 ProMicro, U2 ProMicro

Commit message: moved almost everything into the new jade directory
Parts:
- removed the G*** at (502.5, 165.1)
- removed the G*** at (502.7, 165.1)
- removed the Ref** at (421.1, 166.9)
- removed the Ref** at (432.1, 157.7)
- removed the Ref** at (530.9, 129.3)
- removed the Ref** at (455.0, 125.8)
- removed the Ref** at (502.4, 168.5)
- removed the Ref** at (453.1, 167.9)
- removed the Ref** at (532.2, 166.5)
- removed the SW22 at (540.5, 119.8)
- removed the SW23 at (521.5, 119.8)
- removed the SW24 at (502.5, 115.1)
- removed the SW25 at (483.5, 112.7)
- removed the SW26 at (464.5, 115.1)
- removed the SW27 at (445.5, 117.5)
- removed the SW28 at (540.5, 138.8)
- removed the SW29 at (521.5, 138.8)
- removed the SW30 at (502.5, 134.1)
- removed the SW31 at (483.5, 131.7)
- removed the SW32 at (464.5, 134.1)
- removed the SW33 at (445.5, 136.5)
- removed the SW34 at (540.5, 157.8)
- removed the SW35 at (521.5, 157.8)
- removed the SW36 at (502.5, 153.1)
- removed the SW37 at (483.5, 150.7)
- removed the SW38 at (464.5, 153.1)
- removed the SW39 at (445.5, 155.5)
- removed the SW40 at (465.4, 175.8)
- removed the SW41 at (454.3, 197.2)
- removed the SW42 at (445.8, 179.9)
- removed the SW46 at (535.7, 176.9)
- removed the SW47 at (516.6, 176.9)
- removed the SW48 at (488.0, 172.2)
Routing:
- net VDD: track 660.7 -> 652.6 mm
- net col2_r: track 160.0 -> 156.7 mm
- net GNDA: track 725.1 -> 724.8 mm, vias 17 -> 16
- net Net-(LED47-Pad4): vias 2 -> 4
Other:
- board size 539 x 198.5 mm -> 275.5 x 114.5 mm

Commit message: added logos on silkscreen and plotted all gerber files again
Parts:
- removed the G*** at (238.6, 81.0)
- removed the G*** at (238.8, 81.0)
- removed the G*** at (58.0, 80.9)
- removed the G*** at (58.3, 80.9)
- added G***: LOGO, logo:jdkbd-logo2, F.Cu at (43.2, 83.6)
- added G***: LOGO, logo:jdkbd-logo2, F.Cu at (253.9, 83.6)
Other:
- board text added: "https://github.com/JannikWibker based on crkbd"
- board text added: "jdkbd pcb - designed by jannikwibker"
- board text removed: "cornetrack pcb - designed by jannikwibker"

Commit message: moved tracks further away from edges
Routing:
- net row0: track 220.9 -> 191.2 mm
- net GNDA: track 724.8 -> 701.4 mm, vias 16 -> 19
- net row0_r: track 193.6 -> 187.8 mm
- net row1_r: track 180.7 -> 175.4 mm
- net GND: track 718.8 -> 713.8 mm, vias 22 -> 24
- net row2_r: track 185.2 -> 180.4 mm
- net LED: track 45.0 -> 40.2 mm
- net row1: track 199.1 -> 195.9 mm
- net VCC: track 597.7 -> 595.8 mm
- net col4: track 141.5 -> 140.4 mm
- net Net-(LED56-Pad4): track 48.8 -> 48.0 mm
